File: Eagle/doubleSocket/Double Socket_ESP-12.sch (EAGLE design)
At the start: 29 parts, among them IC1 LM1117IMPX-3.3, K1 G5L, K2 G5L, T1 2N3904, T2 2N3904

Commit message: temp version
Parts:
- removed C1: 100, rcl:CPOL-EUE5-10.5
- removed C2: 1000, rcl:CPOL-EUE5-10.5
- added C3: 100uF, rcl:C-USC0805
- added C4: 1000uF, rcl:C-USC0805
- added U$1: HLK-PM01, aobotelhoLibrary:HLK-PM01
Connections:
- net N$10 renamed OPTO_LED-1
- net N$3 renamed OPTO_LED+2
- net N$4 renamed OPT_EMITTER2
- net N$5 renamed OPT_LED-2
- net N$6 renamed OPTO_LED+1
- net N$9 renamed OPTO_EMITTER1
- removed net N$1: K12.P, X1-2.KL
- removed net N$15: K22.P, X2-2.KL
- new net AC1: K12.P, K22.P, U$1.AC1, X3-2.KL
- new net AC2: U$1.AC2, X1-2.KL, X2-2.KL, X3-1.KL
- net 5V: now also C3.1, U$1.VO+; no longer C1.+, X3-2.KL
- net GND: now also C3.2, C4.2, U$1.VO-; no longer C1.-, C2.-, X3-1.KL
- net VCC: now also C4.1; no longer C2.+
Other:
- moved on the sheet: X3-1, X3-2
Changed lines of the file:
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@@
 <part name="K1" library="relay" deviceset="G5L" device=""/>
 <part name="IC1" library="lm1117" deviceset="LM1117IMPX-*" device="" technology="3.3"/>
-<part name="C1" library="rcl" deviceset="CPOL-EU" device="E5-10.5" value="100"/>
-<part name="C2" library="rcl" deviceset="CPOL-EU" device="E5-10.5" value="1000"/>
 <part name="GND3" library="supply1" library_urn="urn:adsk.eagle:library:371" deviceset="GND" device=""/>
 <part name="P+5" library="supply1" library_urn="urn:adsk.eagle:library:371" deviceset="VCC" device=""/>
@@
 <part name="P+9" library="supply1" library_urn="urn:adsk.eagle:library:371" deviceset="VCC" device=""/>
 <part name="P+10" library="supply1" library_urn="urn:adsk.eagle:library:371" deviceset="VCC" device=""/>
+<part name="C3" library="rcl" deviceset="C-US" device="C0805" value="100uF"/>
+<part name="C4" library="rcl" deviceset="C-US" device="C0805" value="1000uF"/>
+<part name="U$1" library="aobotelhoLibrary" deviceset="HLK-PM01" device=""/>
 </parts>
 <sheets>
@@
 <instance part="K1" gate="2" x="-58.42" y="12.7" rot="R270"/>
 <instance part="IC1" gate="G$1" x="-83.82" y="124.46"/>
-<instance part="C1" gate="G$1" x="-99.06" y="119.38"/>
-<instance part="C2" gate="G$1" x="-68.58" y="121.92"/>
 <instance part="GND3" gate="1" x="-83.82" y="109.22"/>
-<instance part="P+5" gate="VCC" x="-68.58" y="127"/>
+<instance part="P+5" gate="VCC" x="-68.58" y="132.08"/>
 <instance part="OK1" gate="A" x="-106.68" y="5.08"/>
 <instance part="R5" gate="G$1" x="-124.46" y="7.62"/>
@@
 <instance part="X2" gate="-1" x="-40.64" y="53.34" rot="MR0"/>
 <instance part="X2" gate="-2" x="-40.64" y="45.72" rot="MR0"/>
-<instance part="X3" gate="-1" x="-104.14" y="111.76" rot="MR180"/>
-<instance part="X3" gate="-2" x="-104.14" y="124.46" rot="MR180"/>
+<instance part="X3" gate="-1" x="-167.64" y="119.38" rot="MR180"/>
+<instance part="X3" gate="-2" x="-167.64" y="124.46" rot="MR180"/>
 <instance part="X4" gate="-1" x="-5.08" y="25.4" rot="MR0"/>
 <instance part="X4" gate="-2" x="-5.08" y="20.32" rot="MR0"/>
@@
 <instance part="P+9" gate="VCC" x="-139.7" y="88.9"/>
 <instance part="P+10" gate="VCC" x="-66.04" y="96.52"/>
+<instance part="C3" gate="G$1" x="-99.06" y="119.38"/>
+<instance part="C4" gate="G$1" x="-68.58" y="119.38"/>
+<instance part="U$1" gate="G$1" x="-134.62" y="121.92"/>
 </instances>
 <busses>
@@
 <pinref part="GND3" gate="1" pin="GND"/>
 <wire x1="-83.82" y1="111.76" x2="-83.82" y2="116.84" width="0.1524" layer="91"/>
-<pinref part="C2" gate="G$1" pin="-"/>
 <wire x1="-83.82" y1="111.76" x2="-68.58" y2="111.76" width="0.1524" layer="91"/>
-<wire x1="-68.58" y1="111.76" x2="-68.58" y2="116.84" width="0.1524" layer="91"/>
-<pinref part="C1" gate="G$1" pin="-"/>
+<wire x1="-68.58" y1="111.76" x2="-68.58" y2="114.3" width="0.1524" layer="91"/>
+<pinref part="C4" gate="G$1" pin="2"/>
+<pinref part="C3" gate="G$1" pin="2"/>
 <wire x1="-99.06" y1="111.76" x2="-99.06" y2="114.3" width="0.1524" layer="91"/>
-<pinref part="X3" gate="-1" pin="KL"/>
 <wire x1="-99.06" y1="111.76" x2="-83.82" y2="111.76" width="0.1524" layer="91"/>
+<pinref part="U$1" gate="G$1" pin="VO-"/>
+<wire x1="-121.92" y1="119.38" x2="-121.92" y2="111.76" width="0.1524" layer="91"/>
+<wire x1="-121.92" y1="111.76" x2="-99.06" y2="111.76" width="0.1524" layer="91"/>
 </segment>
 <segment>
@@
 <segment>
 <pinref part="IC1" gate="G$1" pin="OUT"/>
-<pinref part="C2" gate="G$1" pin="+"/>
+<wire x1="-68.58" y1="129.54" x2="-68.58" y2="124.46" width="0.1524" layer="91"/>
 <wire x1="-68.58" y1="124.46" x2="-76.2" y2="124.46" width="0.1524" layer="91"/>
 <pinref part="P+5" gate="VCC" pin="VCC"/>
-<junction x="-68.58" y="124.46"/>
 <pinref part="IC1" gate="G$1" pin="OUT1"/>
 <wire x1="-76.2" y1="127" x2="-76.2" y2="124.46" width="0.1524" layer="91"/>
+<pinref part="C4" gate="G$1" pin="1"/>
+<wire x1="-68.58" y1="121.92" x2="-68.58" y2="124.46" width="0.1524" layer="91"/>
 </segment>
 <segment>
@@
 <segment>
 <label x="-99.06" y="124.46" size="1.778" layer="95"/>
-<pinref part="C1" gate="G$1" pin="+"/>
 <wire x1="-99.06" y1="121.92" x2="-99.06" y2="124.46" width="0.1524" layer="91"/>
-<pinref part="X3" gate="-2" pin="KL"/>
+<pinref part="C3" gate="G$1" pin="1"/>
 <pinref part="IC1" gate="G$1" pin="IN"/>
-<wire x1="-91.44" y1="124.46" x2="-99.06" y2="124.46" width="0.1524" layer="91"/>
+<wire x1="-99.06" y1="124.46" x2="-91.44" y2="124.46" width="0.1524" layer="91"/>
+<pinref part="U$1" gate="G$1" pin="VO+"/>
+<wire x1="-99.06" y1="124.46" x2="-121.92" y2="124.46" width="0.1524" layer="91"/>
 </segment>
 <segment>
@@
 </segment>
 </net>
-<net name="N$1" class="0">
-<segment>
-<pinref part="K1" gate="2" pin="P"/>
-<pinref part="X1" gate="-2" pin="KL"/>
-<wire x1="-45.72" y1="10.16" x2="-45.72" y2="2.54" width="0.1524" layer="91"/>
-<wire x1="-45.72" y1="2.54" x2="-60.96" y2="2.54" width="0.1524" layer="91"/>
-<wire x1="-60.96" y1="2.54" x2="-60.96" y2="12.7" width="0.1524" layer="91"/>
-</segment>
-</net>
 <net name="N$2" class="0">
 <segment>
@@
 </segment>
 </net>
-<net name="N$3" class="0">
+<net name="OPTO_LED+2" class="0">
 <segment>
 <pinref part="OK1" gate="A" pin="A"/>
@@
 </segment>
 </net>
-<net name="N$4" class="0">
+<net name="OPT_EMITTER2" class="0">
 <segment>
 <pinref part="OK1" gate="A" pin="EMIT"/>
@@
 </segment>
 </net>
-<net name="N$5" class="0">
+<net name="OPT_LED-2" class="0">
 <segment>
 <pinref part="OK1" gate="A" pin="C"/>
@@
 </segment>
 </net>
-<net name="N$6" class="0">
+<net name="OPTO_LED+1" class="0">
 <segment>
 <pinref part="OK2" gate="A" pin="A"/>
@@
 </segment>
 </net>
-<net name="N$9" class="0">
+<net name="OPTO_EMITTER1" class="0">
 <segment>
 <pinref part="OK2" gate="A" pin="EMIT"/>
@@
 </segment>
 </net>
-<net name="N$10" class="0">
+<net name="OPTO_LED-1" class="0">
 <segment>
 <pinref part="OK2" gate="A" pin="C"/>
@@
 </segment>
 </net>
-<net name="N$15" class="0">
-<segment>
-<pinref part="K2" gate="2" pin="P"/>
-<pinref part="X2" gate="-2" pin="KL"/>
-<wire x1="-45.72" y1="45.72" x2="-45.72" y2="38.1" width="0.1524" layer="91"/>
-<wire x1="-45.72" y1="38.1" x2="-60.96" y2="38.1" width="0.1524" layer="91"/>
-<wire x1="-60.96" y1="38.1" x2="-60.96" y2="48.26" width="0.1524" layer="91"/>
-</segment>
-</net>
 <net name="INPUT2" class="0">
 <segment>
@@
 </segment>
 </net>
+<net name="AC1" class="0">
+<segment>
+<pinref part="U$1" gate="G$1" pin="AC1"/>
+<pinref part="X3" gate="-2" pin="KL"/>
+<wire x1="-162.56" y1="124.46" x2="-147.32" y2="124.46" width="0.1524" layer="91"/>
+</segment>
+<segment>
+<pinref part="K2" gate="2" pin="P"/>
+<wire x1="-60.96" y1="38.1" x2="-60.96" y2="48.26" width="0.1524" layer="91"/>
+<label x="-60.96" y="38.1" size="1.778" layer="95" rot="R90"/>
+</segment>
+<segment>
+<pinref part="K1" gate="2" pin="P"/>
+<wire x1="-60.96" y1="2.54" x2="-60.96" y2="12.7" width="0.1524" layer="91"/>
+<label x="-60.96" y="2.54" size="1.778" layer="95" rot="R90"/>
+</segment>
+</net>
+<net name="AC2" class="0">
+<segment>
+<pinref part="U$1" gate="G$1" pin="AC2"/>
+<pinref part="X3" gate="-1" pin="KL"/>
+<wire x1="-162.56" y1="119.38" x2="-147.32" y2="119.38" width="0.1524" layer="91"/>
+</segment>
+<segment>
+<pinref part="X2" gate="-2" pin="KL"/>
+<wire x1="-45.72" y1="45.72" x2="-45.72" y2="38.1" width="0.1524" layer="91"/>
+<label x="-45.72" y="38.1" size="1.778" layer="95" rot="R90"/>
+</segment>
+<segment>
+<pinref part="X1" gate="-2" pin="KL"/>
+<wire x1="-45.72" y1="10.16" x2="-45.72" y2="2.54" width="0.1524" layer="91"/>
+<label x="-45.72" y="2.54" size="1.778" layer="95" rot="R90"/>
+</segment>
+</net>
